Commit message: feat: v2 training pipeline — multi-view, domain randomization, resnet50, real fine-tuning
URDF — Multi-Camera:
- Added 3 additional camera viewpoints (right, left, top) alongside
  existing front camera → 4 total views for multi-view training
- Camera positions: front (0.8,0,0.4), right (0,0.8,0.4),
  left (0,-0.8,0.4), top (0,0,1.2)

Domain Randomization:
- New Gazebo world: worlds/randomized.sdf with varied lighting
  (directional sun, fill light, warm point light), ground plane,
  back wall, side panel, table, and 3 clutter objects
- Collector v2 randomizes sun direction/color and point light
  position per sample via gz service calls
- Per-image Gaussian noise injection (configurable σ)

Data Collection v2:
- synthetic_data_collector_v2.py: multi-camera capture, domain
  randomization, noise injection, CSV with camera column
- synthetic_data_v2.launch.py: launches randomized world + 4 camera
  bridges + enhanced collector
- Default 5000 samples, 85% joint range

Training Pipeline v2:
- dataset.py: MyCobotMultiViewDataset (groups views per pose),
  MergedPoseDataset (synthetic+real), camera_filter for single-view
  from multi-view CSV, heavier augmentation (RandomAffine, RandomErasing)
- model.py: MultiViewPoseResNet with shared backbone + fusion MLP,
  extract_features() method for feature analysis
- train.py: --multi-view, --real-dataset (merge), --finetune,
  --camera-filter, --num-views flags; _TransformSubsetMV for
  multi-view data; fine-tune mode with auto freeze-epochs

Real Data Capture:
- training/capture_real.py: TCP bridge + OpenCV capture utility,
  produces same CSV format for seamless fine-tuning

ResNet50 benchmark (1000 samples): 20.9° mean MAE vs 22.6° resnet18

File: mycobot_description/urdf/320_pi/mycobot_pro_320_pi_gazebo.urdf (robot description, URDF)
Before this commit: robot mycobot_320_pi, 9 links, 8 joints
Links:
- added link camera_link_left, mass 0.01; visual box size=0.03 0.03 0.03
- added link camera_link_right, mass 0.01; visual box size=0.03 0.03 0.03
- added link camera_link_top, mass 0.01; visual box size=0.03 0.03 0.03
Joints:
- added joint world_to_camera_left: type fixed, parent world, child camera_link_left, origin xyz=0.0 -0.8 0.4 rpy=0 0.3 1.5708
- added joint world_to_camera_right: type fixed, parent world, child camera_link_right, origin xyz=0.0 0.8 0.4 rpy=0 0.3 -1.5708
- added joint world_to_camera_top: type fixed, parent world, child camera_link_top, origin xyz=0.0 0.0 1.2 rpy=0 1.5708 0

Commit message: feat: gripper integration, v2 data pipeline, and full docs update
- Add pro_adaptive_gripper meshes + link6_2022.dae (gripper compat.)
- Add worlds/randomized_v2.sdf (6 lights, 12 clutter objects, 3 walls)
- Add synthetic_data_v3.launch.py (randomized_v2 world)
- Add anti-collision FK filtering in synthetic_data_collector_v2.py
- Add merge_and_convert.py (real+synth dataset merge with oversampling)
- Add finetune_real.py (experimental — documented as non-functional)
- Add train_pipeline.sh and monitor_collection.sh utility scripts
- Fix joint limits in gazebo URDF (J2: ±134.6°, J3/J4: ±145.0°)
- Rewrite SESSION_RESUME.md (was a corrupted merge artifact)
- Update CHANGELOG.md with full version history (v0.1.0 → v1.9.0)
- Update all README and docs to reflect April 2026 project state:
  fix stale IP (10.10.0.218 → 10.10.0.225), remove "en cours" markers,
  add missing files to project structure, update sim-to-real results

File: mycobot_description/urdf/320_pi/mycobot_pro_320_pi_gazebo.urdf (robot description, URDF)
Before this commit: robot mycobot_320_pi, 12 links, 11 joints
Links:
- added link gripper_base, mass 0.1; collision mesh filename=package://mycobot_description/urdf/pro_adaptive_gripper/gri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; visual mesh filename=package://mycobot_description/urdf/pro_adaptive_gripper/gri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
- added link gripper_left1, mass 0.02; collision mesh filename=package://mycobot_description/urdf/pro_adaptive_gripper/gri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; visual mesh filename=package://mycobot_description/urdf/pro_adaptive_gripper/gri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
- added link gripper_left2, mass 0.02; collision mesh filename=package://mycobot_description/urdf/pro_adaptive_gripper/gri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; visual mesh filename=package://mycobot_description/urdf/pro_adaptive_gripper/gri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
- added link gripper_left3, mass 0.02; collision mesh filename=package://mycobot_description/urdf/pro_adaptive_gripper/gri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; visual mesh filename=package://mycobot_description/urdf/pro_adaptive_gripper/gri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
- added link gripper_right1, mass 0.02; collision mesh filename=package://mycobot_description/urdf/pro_adaptive_gripper/gri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; visual mesh filename=package://mycobot_description/urdf/pro_adaptive_gripper/gri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
- added link gripper_right2, mass 0.02; collision mesh filename=package://mycobot_description/urdf/pro_adaptive_gripper/gri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; visual mesh filename=package://mycobot_description/urdf/pro_adaptive_gripper/gri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
- added link gripper_right3, mass 0.02; collision mesh filename=package://mycobot_description/urdf/pro_adaptive_gripper/gri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; visual mesh filename=package://mycobot_description/urdf/pro_adaptive_gripper/gri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
- link link6: geometry collision mesh filename=package://mycobot_description/urdf/320_pi/link6_2022.dae; visual mesh filename=package://mycobot_description/urdf/320_pi/link6_2022.dae
Joints:
- added joint gripper_base_to_gripper_left2: type fixed, parent gripper_base, child gripper_left2, origin xyz=-0.047 -0.01 0 rpy=0 0 0
- added joint gripper_base_to_gripper_right2: type fixed, parent gripper_base, child gripper_right2, origin xyz=0.044 -0.01 0 rpy=0 0 0
- added joint gripper_base_to_gripper_right3: type fixed, parent gripper_base, child gripper_right3, origin xyz=0.016 0.014 0 rpy=0 0 0
- added joint gripper_controller: type fixed, parent gripper_base, child gripper_left3, origin xyz=-0.018 0.015 0 rpy=0 0 0
- added joint gripper_left3_to_gripper_left1: type fixed, parent gripper_left3, child gripper_left1, origin xyz=-0.05 0.035 -0.015 rpy=0 0 0
- added joint gripper_right3_to_gripper_right1: type fixed, parent gripper_right3, child gripper_right1, origin xyz=0.052 0.035 -0.015 rpy=0 0 0
- added joint joint6output_to_gripper_base: type fixed, parent link6, child gripper_base, origin xyz=0.0 -0.007 0.056 rpy=1.5708 0 0
- joint joint2_to_joint1: limit lower=-2.96 upper=2.96 effort=1000.0 velocity=3.14 -> lower=-2.93 upper=2.93 effort=1000.0 velocity=3.14
- joint joint3_to_joint2: limit lower=-2.79 upper=2.79 effort=1000.0 velocity=3.14 -> lower=-2.35 upper=2.35 effort=1000.0 velocity=3.14
- joint joint4_to_joint3: limit lower=-2.79 upper=2.79 effort=1000.0 velocity=3.14 -> lower=-2.53 upper=2.53 effort=1000.0 velocity=3.14
- joint joint5_to_joint4: limit lower=-2.79 upper=2.79 effort=1000.0 velocity=3.14 -> lower=-2.53 upper=2.53 effort=1000.0 velocity=3.14
- joint joint6_to_joint5: limit lower=-2.96 upper=2.96 effort=1000.0 velocity=3.14 -> lower=-2.93 upper=2.93 effort=1000.0 velocity=3.14
- joint joint6output_to_joint6: limit lower=-3.05 upper=3.05 effort=1000.0 velocity=3.14 -> lower=-3.14 upper=3.14 effort=1000.0 velocity=3.14

Commit message: feat(gripper): make adaptive gripper functional in Gazebo sim
URDF:
- gripper_controller joint goes from fixed to revolute (axis=z,
  limit -0.7..0 rad, velocity 3.14) — drives the left finger stack
- gripper_base_to_gripper_right3 also revolute + <mimic> pointing to
  gripper_controller with multiplier=-1 (mirrors the right finger)
- Finger-tip joints (left1, left2, right1, right2) stay fixed; the
  visual articulation is carried by the two servo joints, which is
  enough to see a clear open/close motion in Gazebo
- Added matching <joint> blocks inside the <ros2_control> system:
  gripper_controller has position command + position/velocity state;
  gripper_base_to_gripper_right3 is declared with mimic/multiplier
  params so gz_ros2_control replicates the motion

controller.yaml:
- Added a gripper_position_controller
  (position_controllers/JointGroupPositionController) with one joint
  (gripper_controller) and conservative PID gains + antiwindup

Launch:
- Spawner for gripper_position_controller, staggered 0.5 s after the
  arm controller so they don't race on the controller manager

teleop/mycobot_teleop.py:
- RosBridgeArmPublisher advertises /gripper_position_controller/commands
  and exposes send_gripper_normalized(openness∈[0,1]) that maps to the
  URDF range (-0.7 rad closed → 0 rad open)
- Main loop now extracts pose.open_degree from Wilor and normalizes it
  via SAFE_RANGE["g"] = (2, 90) before sending

Tested: URDF still parses (669 lines, mimic tags present), colcon build
succeeds for both mycobot_description and mycobot_gateway.

File: mycobot_description/urdf/320_pi/mycobot_pro_320_pi_gazebo.urdf (robot description, URDF)
Before this commit: robot mycobot_320_pi, 19 links, 18 joints
Joints:
- joint gripper_base_to_gripper_right3: axis (none) -> 0 0 1; limit (none) -> lower=0.0 upper=0.7 effort=10.0 velocity=3.14; mimic (none) -> joint=gripper_controller multiplier=-1.0 offset=0.0; type fixed -> revolute
- joint gripper_controller: axis (none) -> 0 0 1; limit (none) -> lower=-0.7 upper=0.0 effort=10.0 velocity=3.14; type fixed -> revolute

Commit message: fix(gripper): 4-bar linkage — fingertips stay parallel to gripper base
The first gripper revision only unfroze the two servo joints
(gripper_controller → left3, gripper_base_to_gripper_right3 → right3).
The fingertip joints (left3→left1, right3→right1) stayed fixed, so the
finger blades rotated rigidly with their pivots — producing the splayed,
non-parallel closure visible in the user's screenshots (the right fingertip
swinging outward instead of translating toward the left one).

URDF can't express closed kinematic loops, so the real adaptive gripper's
4-bar linkage isn't reproducible exactly. Approximation: unfreeze both
tip joints and mimic gripper_controller with multipliers that counter-
rotate them exactly opposite to their parent, so the fingertip frames
stay aligned with gripper_base throughout the servo sweep.

    gripper_left3_to_gripper_left1:
        mimic(gripper_controller, multiplier=-1)
        → left1 relative to left3 = -θ_servo, absolute = 0

    gripper_right3_to_gripper_right1:
        mimic(gripper_controller, multiplier=+1)
        → right3 already at +θ (it itself mimics -1), right1 relative
          = +θ_servo, absolute = 0 as well

Also added both joints to the <ros2_control> block with matching mimic
params + state interfaces so gz_ros2_control writes them at each hardware
cycle (DART physics ignores the URDF <mimic> constraint natively, but the
ros2_control plugin honours it at the state interface level).

URDF still parses: 700 lines, 5 <mimic> tags.

File: mycobot_description/urdf/320_pi/mycobot_pro_320_pi_gazebo.urdf (robot description, URDF)
Before this commit: robot mycobot_320_pi, 19 links, 18 joints
Joints:
- joint gripper_left3_to_gripper_left1: axis (none) -> 0 0 1; limit (none) -> lower=-0.7 upper=0.7 effort=2.0 velocity=3.14; mimic (none) -> joint=gripper_controller multiplier=-1.0 offset=0.0; type fixed -> revolute
- joint gripper_right3_to_gripper_right1: axis (none) -> 0 0 1; limit (none) -> lower=-0.7 upper=0.7 effort=2.0 velocity=3.14; mimic (none) -> joint=gripper_controller multiplier=1.0 offset=0.0; type fixed -> revolute

Commit message: fix(gripper): drive the 4 gripper joints explicitly, no mimic
Root cause of the droop: gz_ros2_control only loads joints that appear
in the <ros2_control> block. In the previous revision the mimic
fingertip joints were declared only in the URDF <joint><mimic> form,
not in <ros2_control>, so gz_ros2_control never saw them. DART physics
doesn't enforce URDF mimic constraints either (Physics.cc logs
"the chosen physics engine does not support mimic constraints"), so
those joints were left as free-floating revolutes and gravity ruled.

Giving them command_interfaces crashed controller_manager:
    "Activated mimic joints cannot have command interfaces"

So the escape is to drop URDF mimic entirely and command all four
gripper joints from a single JointGroupPositionController. The
mycobot_teleop.py helper publishes a 4-element array with the
appropriate signs to keep the gripper mirrored and the fingertips
parallel to the base:

    open  (o=1):  [ 0, 0, 0, 0 ]
    close (o=0):  [ -0.7, +0.7, +0.7, -0.7 ]

Changes:
- URDF: removed <mimic> tags from gripper_base_to_gripper_right3,
  gripper_left3_to_gripper_left1, gripper_right3_to_gripper_right1
  (all three stay revolute with the same limits).
- URDF: added the three joints to <ros2_control> with position
  command_interfaces + state_interfaces.
- controller.yaml: gripper_position_controller now lists all four
  joints; tips run on softer PID (p=30) than the servos (p=60).
- mycobot_teleop.py: send_gripper_normalized publishes the 4-element
  symmetric array described above.

With this the gripper should open / close symmetrically AND the
fingertips should stay parallel to gripper_base — matching the real
adaptive gripper's 4-bar kinematics visually, without needing URDF
closed-loop support.

File: mycobot_description/urdf/320_pi/mycobot_pro_320_pi_gazebo.urdf (robot description, URDF)
Before this commit: robot mycobot_320_pi, 19 links, 18 joints
Joints:
- joint gripper_base_to_gripper_right3: mimic joint=gripper_controller multiplier=-1.0 offset=0.0 -> (none)
- joint gripper_left3_to_gripper_left1: mimic joint=gripper_controller multiplier=-1.0 offset=0.0 -> (none)
- joint gripper_right3_to_gripper_right1: mimic joint=gripper_controller multiplier=1.0 offset=0.0 -> (none)

Commit message: feat(sorting): multi-object color pick-and-place + camera reshape
New: pick-and-place sorting pipeline that picks 4 colored objects
(red cube, blue cube, green cylinder, yellow box) and drops each
into its color-matching bin. Extends the existing single-object
pick-and-place foundation (IK solver, joint command bridge) with
HSV-based perception and a multi-target orchestrator.

Components:
- worlds/pick_and_place_sorting.sdf: 1.0x0.6 m table, 4 dynamic
  objects on +X side, 4 walled colored bins on -X side, all inside
  the ~0.32 m MyCobot 320 reach envelope.
- color_object_detector.py: HSV segmentation on the top-down camera
  with pinhole back-projection to robot-frame XY. Publishes
  /sorting/detections, /sorting/detector_status, /sorting/debug_image.
- sorting_orchestrator.py: state machine that loops over detections,
  plans IK per target, and emulates grasp/release via the gz
  /world/<world>/set_pose service (object follows EE during carry,
  drops at bin XY at release).
- launch/pick_and_place_sorting.launch.py: Gazebo + spawn + bridges
  + 4 cameras + detector (T+6 s) + orchestrator (T+10 s).
  Args: use_detector, process_order.

URDF camera reshape:
The 4 onboard cameras were 3 cm colored cubes that visually clashed
with the colored sort objects. Replaced each with a real-camera
silhouette: dark-gray body box (0.06x0.04x0.04) + black lens
cylinder along the optical axis (+X) + tiny red LED. Sensor poses
unchanged.

Bug fixes surfaced during live test:
- color_object_detector params 'image_u_to_world_axis' / '..._v_...'
  defaulted to 'y' / 'x', which YAML 1.1 coerces to bool True. rclpy
  rejected the param. Renamed to *_axis_name with 'world_y' /
  'world_x' values.
- Top-camera Y axis was sign-flipped (red detected at +0.12 instead
  of -0.12). Set flip_u: True in the launch file. Verified live:
  detector positions now match SDF ground truth to ~1 mm.

Verified end-to-end on this branch: 4 colors sorted in ~95 s,
no IK failures, no set_pose failures, all objects land in the
correct bin.

Docs updated: CHANGELOG (1.10.0), SESSION_RESUME (branch + activity
table + commands), README (new launch + sorting subsection),
docs/ARCHITECTURE (nodes, launches, worlds, camera visuals),
mycobot_gateway/README (nodes, launches, topics), README_GAZEBO
(new worlds + camera-visual rationale).

File: mycobot_description/urdf/320_pi/mycobot_pro_320_pi_gazebo.urdf (robot description, URDF)
Before this commit: robot mycobot_320_pi, 19 links, 18 joints
Links:
- link camera_link: geometry visual box size=0.06 0.04 0.04; visual cylinder length=0.025 radius=0.013
- link camera_link_left: geometry visual box size=0.06 0.04 0.04; visual cylinder length=0.025 radius=0.013
- link camera_link_right: geometry visual box size=0.06 0.04 0.04; visual cylinder length=0.025 radius=0.013
- link camera_link_top: geometry visual box size=0.06 0.04 0.04; visual cylinder length=0.025 radius=0.013
