Commit message: feat: natural lighting world + headless pipeline for 50k acquisition
- Add lab_room.sdf: 3-light warm/cool setup, SDF 1.6, world name 'empty'
- Fix URDF XML comments (-- forbidden inside <!-- -->)
- Add synthetic_data_preview.launch.py (5 poses visual check)
- Both launch files use lab_room.sdf + -s --headless-rendering
- setup.py installs worlds/*.sdf

Co-Authored-By: Claude Sonnet 4.6 <noreply@anthropic.com>

File: mycobot_description/urdf/320_pi/mycobot_pro_320_pi_gazebo.urdf (robot description, URDF)
Before this commit: robot mycobot_320_pi, 9 links, 8 joints
Links:
- added link camera_link_1, mass 0.01; visual box size=0.03 0.03 0.03
- added link camera_link_2, mass 0.01; visual box size=0.03 0.03 0.03
- added link camera_link_3, mass 0.01; visual box size=0.03 0.03 0.03
Joints:
- added joint world_to_camera_1: type fixed, parent world, child camera_link_1, origin xyz=0.0 0.8 0.4 rpy=0 0.30 -1.5708
- added joint world_to_camera_2: type fixed, parent world, child camera_link_2, origin xyz=-0.7 0.0 0.4 rpy=0 0.50 0.0
- added joint world_to_camera_3: type fixed, parent world, child camera_link_3, origin xyz=0.0 -0.8 0.4 rpy=0 0.30 1.5708
- joint world_to_camera: origin xyz=0.8 0.0 0.4 rpy=0 0.3 3.1416 -> xyz=0.8 0.0 0.4 rpy=0 0.30 3.1416

Commit message: fix(gazebo): une seule convention de nom pour les 3 cameras secondaires
Le depot en portait deux. Le URDF publiait synth_camera_1/2/3, alors que
pick_and_place, pick_and_place_sorting, synthetic_data_v2, synthetic_data_v3,
color_object_detector et synthetic_data_collector_v2 s'abonnaient deja a
right/left/top -- donc a rien, puisque aucun world .sdf ne definit de camera.
Les noms de joints (world_to_camera_right/left/top) et README_GAZEBO.md
etaient eux aussi du cote right/left/top : le _1/2/3 etait l'exception.

Le correctif du 10/09 (a9df378e) avait reparee le parsing URDF en alignant
les liens sur _1/2/3, c'est-a-dire du mauvais cote de la scission -- il
rendait le robot chargeable sans rendre les topics joignables.

Renomme donc les liens, les capteurs et les topics en right/left/top, et
recable les trois seuls utilisateurs de l'ancienne convention
(synthetic_data.launch.py, synthetic_data_preview.launch.py,
synthetic_data_collector.py).

Le cablage physique du collecteur v1 ne change pas : cam_1 reste la camera
du cote +Y, cam_2 celle du cote -Y, cam_3 la zenithale. Son commentaire
appelait cam_1 « left », ce que contredisaient a la fois le nom du joint et
le collecteur v2 ; remplace par la position geometrique, qui ne suppose
aucune convention. Quel cote merite le nom « droite » reste ouvert.

Verifie : URDF bien forme, aucun joint ne reference un lien inexistant,
plus aucune occurrence de l'ancienne convention hors entrees datees.

Co-Authored-By: Claude Opus 5 <noreply@anthropic.com>

File: mycobot_description/urdf/320_pi/mycobot_pro_320_pi_gazebo.urdf (robot description, URDF)
Before this commit: robot mycobot_320_pi, 19 links, 18 joints
Links:
- removed link camera_link_1
- removed link camera_link_2
- removed link camera_link_3
- added link camera_link_left, mass 0.01; visual box size=0.03 0.03 0.03
- added link camera_link_right, mass 0.01; visual box size=0.03 0.03 0.03
- added link camera_link_top, mass 0.01; visual box size=0.03 0.03 0.03
Joints:
- joint world_to_camera_left: child camera_link_2 -> camera_link_left
- joint world_to_camera_right: child camera_link_1 -> camera_link_right
- joint world_to_camera_top: child camera_link_3 -> camera_link_top

Commit message: feat(gazebo): tri des 4 pieces pilote par yolo26 sur 4 cameras
La scene tri_yolo place 4 pieces et 4 bacs sur la replique du banc, vue
par les 4 cameras du jeu DREAM 50K. Le bras simule trie a partir de la
perception seule : yolo26 v6c sur chaque camera, boite 3D de la classe
recalee sur la boite 2D, fusion par la mediane des cameras (0,65 mm
median, 2,07 mm au pire sur 10 scenes), objet et bac appaires par la
classe. La pose Gazebo ne sert qu'a verifier prise et depot.

sim_sorting_grasp pose_source:=perception : depot resolu avant la
saisie, ouverture d'approche reduite, cubes pinces a 0 ou 90 deg,
largage incline 15/30/45 deg pour les bacs hors de portee verticale,
2 essais apres une prise a vide. Le lacher se fait 5 mm au-dessus du
rebord, doigts ecartes AVANT la remontee : l'objet glissait entre les
doigts, et le cube bleu restait pince par la paroi du bac. Graine 1 :
4/4 tries, chaque objet au fond de son bac.

Spawners avec --switch-timeout 30 : avec 4 cameras rendues,
l'activation depassait parfois les 5 s par defaut.

Detail, mesures et journal : docs/PROTOCOLE_YOLO_GAZEBO.md.

Co-Authored-By: Claude Opus 5.5 <noreply@anthropic.com>

File: mycobot_description/urdf/320_pi/mycobot_pro_320_pi_gazebo.urdf (robot description, URDF)
Before this commit: robot mycobot_320_pi, 19 links, 18 joints
Links:
- removed link camera_link
- removed link camera_link_left
- removed link camera_link_right
- removed link camera_link_top
- link base: mass 0.5 -> None
- link gripper_base: mass 0.1 -> None
- link gripper_left1: mass 0.02 -> None
- link gripper_left2: mass 0.02 -> None
- link gripper_left3: mass 0.02 -> None
- link gripper_right1: mass 0.02 -> None
- link gripper_right2: mass 0.02 -> None
- link gripper_right3: mass 0.02 -> None
- link link1: mass 0.3 -> None
- link link2: mass 0.25 -> None
- link link3: mass 0.2 -> None
- link link4: mass 0.15 -> None
- link link5: mass 0.1 -> None
- link link6: mass 0.08 -> None
Joints:
- removed joint world_to_camera
- removed joint world_to_camera_left
- removed joint world_to_camera_right
- removed joint world_to_camera_top
- joint joint2_to_joint1: limit lower=-2.93 upper=2.93 effort=1000.0 velocity=3.14 -> lower=-2.93215 upper=2.93215 effort=${12.0 if effort_arm else 1000.0} velocity=3.14
- joint joint3_to_joint2: limit lower=-2.35 upper=2.35 effort=1000.0 velocity=3.14 -> lower=-2.35619 upper=2.35619 effort=${12.0 if effort_arm else 1000.0} velocity=3.14
- joint joint4_to_joint3: limit lower=-2.53 upper=2.53 effort=1000.0 velocity=3.14 -> lower=-2.61799 upper=2.61799 effort=${10.0 if effort_arm else 1000.0} velocity=3.14
- joint joint5_to_joint4: limit lower=-2.53 upper=2.53 effort=1000.0 velocity=3.14 -> lower=-2.53073 upper=2.53073 effort=${5.0 if effort_arm else 1000.0} velocity=3.14
- joint joint6_to_joint5: limit lower=-2.93 upper=2.93 effort=1000.0 velocity=3.14 -> lower=-2.87979 upper=2.87979 effort=${4.0 if effort_arm else 1000.0} velocity=3.14
- joint joint6output_to_joint6: limit lower=-3.14 upper=3.14 effort=1000.0 velocity=3.14 -> lower=-3.14159 upper=3.14159 effort=${3.0 if effort_arm else 1000.0} velocity=3.14
