Commit message: feat(pick): pince fiabilisee sur le reel, plugin de commande restaure en sim
REEL — trois defauts de la pince, tous mesures sur le bras.

Une lecture parasite ne fait plus lacher l'objet. Douze lectures tracees
pendant une remontee en trois paliers : deux statuts « 6 » (la pince ne
rend que 0-3) et un angle « 65535 » (le -1 du registre lu en 16 bits non
signes). Une seule suffisait a conclure « objet lache » — la remontee
s'arretait et la pince s'ouvrait EN L'AIR, jetant le rouleau hors de la
planche. `porte_objet` relit jusqu'a trois fois, ignore un temoin
illisible, et repond « tenu » si les deux le restent : croire tenir ce
qu'on ne tient pas coute un cycle, croire avoir lache ce qu'on tient
jette l'objet.

Un statut « objet saisi » sur une pince VIDE ne trompe plus la machine.
Figurine imprimee, roulis 0 : statut 2 avec un angle de 22 — deux degres
au-dessus de la pince vide — et la figurine poussee de 18,3 mm. Conclure
sur le statut seul partait en remontee pour rien ET n'inscrivait jamais
le roulis rate.

Un roulis qui POUSSE n'est plus rejoue (`ctx.prises_ratees`). A 389 mm
seules les inclinaisons -30 et -45 resolvent, et a -30 les roulis 0, 30,
60 et 90 passent tous la geometrie : le roulis 0 referme a vide et pousse
le rouleau de 6,4 mm, le +30 le saisit (statut 2, angle 26) et le tient
jusqu'a Z=170. Le couple rate passe en dernier — ecarte, jamais supprime,
sinon un objet devient insaisissable.

Cycles de tri complets valides : rouleau -> petit carton en 56 s ;
figurine -> grand carton en 73 s, avec rattrapage automatique apres une
premiere saisie perdue. Plateau vide apres coup, verifie camera.

Le seuil vertical/couche passe de 325 a 320 mm, mesure au balayage de
`colonne_continue` (le vertical descend jusqu'a 320, refuse des 324).

SIMULATION — le bras ne bougeait pas du tout. Le plugin
`gz-sim-joint-position-controller-system` avait disparu de l'URDF de
cette copie du depot ; sans lui les topics cmd_pos n'ont aucun abonne,
`ros2 control list_controllers` rend « No controllers are currently
loaded! » et `/joint_states` reste a zero pendant tout le tri. La demo
allait quand meme jusqu'a « Sorting complete » : elle est en boucle
ouverte et TELEPORTE les cubes. Plugin repris tel quel de ~/ros_jazzy.
La demo reste une demo de PLANIFICATION, pas de prehension.

Pince simulee : frottement pose sur les doigts (mu=1,6, ils n'en avaient
aucun alors que les cubes sont a 1,0) et course portee de 0,7 a 1,10 rad
— mesure, les doigts sont a 136 mm au repos et encore 67 mm a 0,7 rad,
trop pour un cube de 40 mm ; a 1,10 ils se referment a 17,9 mm.

Reste ouvert : en simulation `gripper_controller` (servo gauche) ne bouge
jamais quelle que soit la consigne, alors que ses trois voisines suivent
— la pince ne se referme que d'un cote. Et sur le reel, un plafond |J5|
<= 90 deg reste a implementer (mesure : aucune des 120 poses de travail
ne depasse 83 deg, alors que le roulis +90 en demande 121).

File: mycobot_description/urdf/320_pi/mycobot_pro_320_pi_gazebo.urdf (robot description, URDF)
Before this commit: robot mycobot_320_pi, 19 links, 18 joints
Joints:
- joint gripper_base_to_gripper_right3: limit lower=0.0 upper=0.7 effort=10.0 velocity=3.14 -> lower=0.0 upper=1.10 effort=10.0 velocity=3.14
- joint gripper_controller: limit lower=-0.7 upper=0.0 effort=10.0 velocity=3.14 -> lower=-1.10 upper=0.0 effort=10.0 velocity=3.14
- joint gripper_left3_to_gripper_left1: limit lower=-0.7 upper=0.7 effort=2.0 velocity=3.14 -> lower=-1.10 upper=1.10 effort=2.0 velocity=3.14
- joint gripper_right3_to_gripper_right1: limit lower=-0.7 upper=0.7 effort=2.0 velocity=3.14 -> lower=-1.10 upper=1.10 effort=2.0 velocity=3.14
- joint world_to_camera: origin xyz=0.8 0.0 0.4 rpy=0 0.3 3.1416 -> xyz=1.1 0.0 0.4 rpy=0 0.3 3.1416
- joint world_to_camera_left: origin xyz=0.0 -0.8 0.4 rpy=0 0.3 1.5708 -> xyz=0.0 -1.1 0.4 rpy=0 0.3 1.5708
- joint world_to_camera_right: origin xyz=0.0 0.8 0.4 rpy=0 0.3 -1.5708 -> xyz=0.0 1.1 0.4 rpy=0 0.3 -1.5708
- joint world_to_camera_top: origin xyz=0.0 0.0 1.2 rpy=0 1.5708 0 -> xyz=0.0 0.0 1.0 rpy=0 1.5708 0

Commit message: feat(sorting): les quatre objets poses a plat au fond de leur bac
Saisie PHYSIQUE en simulation, sans aucune teleportation : bras au JTC
`mycobot_controller`, pince au `gripper_position_controller`, chaque prise
verifiee sur la pose Gazebo de l'objet. 4/4, les quatre a 0,0 deg
d'inclinaison et au millimetre du fond de leur bac. Cycle en 115 s.

Le point outil est le centre des PATINS, pas le bout des doigts. Viser
l'extremite decale la consigne de 15 mm — la largeur d'un patin. Le cube de
40 mm rattrapait l'erreur par sa largeur, le cylindre de 44 mm non : les
quatre joints atteignaient la consigne au millieme,
preuve de zero contact.

Le poignet ne doit pas tourner entre la saisie et la levee. Resoudre l'IK
independamment a chaque hauteur laissait phi changer d'un point au suivant,
et l'objet se devissait des doigts. `solve_column` impose un phi unique a
survol + saisie + levee.

Le bac vert n'est atteignable que par-dessus l'epaule (J1 = -35 deg, J3 > 0,
J5 < 0) : l'outil sort a ~22 deg d'azimut de J1, donc son azimut de 164,7 deg
demanderait J1 = 187 deg, au-dela de la butee. Vaut aussi pour le vrai bras.

gripper_left2 et gripper_right2 etaient declarees `fixed`, donc soudees a la
bride et fondues dans link6 : immobiles pendant que le doigt tournait, elles
partaient a l'horizontale et la pince paraissait cassee sur les cotes. Ce sont
les barres exterieures d'un quadrilatere articule, paralleles a 0,0 deg pres
a la bielle motrice — un parallelogramme, donc meme angle que le servo.
Passees en revolute et pilotees, le bout reste a 1,0-1,3 mm du doigt sur toute
la course. Le controleur attend desormais 6 valeurs et non 4.

L'objet est pose au fond du bac, plus lache au-dessus. Il tombait de 15 a
25 mm, rebondissait sur la paroi et restait couche sur le rebord (cube bleu a
44,6 deg). La collision doigts/bac demande DEUX conditions simultanees : etre
sous le rebord (30 mm) ET plus ecarte que la paroi interne (+-47,5 mm) — or
refermes les doigts ne font que +-34 a +-44 mm. Lacher en deux temps :
largeur exacte de l'objet, remontee, puis ouverture complete.

Chaque mouvement attendait une duree fixe (4 s + 2,5 s, huit fois par objet).
`move_to` la dimensionne sur le trajet et rend la main des que l'ecart passe
sous 0,35 deg ; l'IK passe de 150 a 60 iterations et s'arrete au premier
resultat franc.

`mycobot_gateway/setup.cfg` manquait : sans lui setuptools installe les points
d'entree dans bin/, ou `ros2 run` ne regarde pas. Tout noeud ajoute au paquet
depuis la migration vers Osama_ws etait introuvable malgre une compilation
reussie.

File: mycobot_description/urdf/320_pi/mycobot_pro_320_pi_gazebo.urdf (robot description, URDF)
Before this commit: robot mycobot_320_pi, 19 links, 18 joints
Joints:
- joint gripper_base_to_gripper_left2: axis (none) -> 0 0 1; limit (none) -> lower=-1.20 upper=0.10 effort=2.0 velocity=3.14; type fixed -> revolute
- joint gripper_base_to_gripper_right2: axis (none) -> 0 0 1; limit (none) -> lower=-0.10 upper=1.20 effort=2.0 velocity=3.14; type fixed -> revolute
- joint gripper_base_to_gripper_right3: limit lower=0.0 upper=1.10 effort=10.0 velocity=3.14 -> lower=-0.10 upper=1.20 effort=10.0 velocity=3.14
- joint gripper_controller: limit lower=-1.10 upper=0.0 effort=10.0 velocity=3.14 -> lower=-1.20 upper=0.10 effort=10.0 velocity=3.14

Commit message: fix(teleop): delayed controller spawners + primitive gripper collisions for gz-physics
- gazebo_sim.launch.py: spawn joint_state_broadcaster/mycobot_controller/
  gripper_position_controller via staggered TimerActions (5/6/7s) so they
  come up after Gazebo has actually spawned the robot entity.
- mycobot_pro_320_pi_gazebo.urdf: replace adaptive-gripper collision meshes
  (.dae) with box primitives and matching inertial origins — gz-physics
  (DART) collision on the fine gripper meshes was unstable/slow. Also
  documents that DART doesn't support <mimic>: left/right finger chains
  are now driven independently by gripper_position_controller with
  opposite-sign commands instead of relying on a mirrored joint.

File: mycobot_description/urdf/320_pi/mycobot_pro_320_pi_gazebo.urdf (robot description, URDF)
Before this commit: robot mycobot_320_pi, 19 links, 18 joints
Links:
- link gripper_base: geometry collision box size=0.1048 0.0434 0.0362; visual mesh filename=package://mycobot_description/urdf/pro_adaptive_gripper/gri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
- link gripper_left1: geometry collision box size=0.0110 0.0055 0.0055; visual mesh filename=package://mycobot_description/urdf/pro_adaptive_gripper/gri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
- link gripper_left2: geometry collision box size=0.0085 0.0085 0.0268; visual mesh filename=package://mycobot_description/urdf/pro_adaptive_gripper/gri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
- link gripper_left3: geometry collision box size=0.0653 0.0435 0.0108; visual mesh filename=package://mycobot_description/urdf/pro_adaptive_gripper/gri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
- link gripper_right1: geometry collision box size=0.0110 0.0055 0.0055; visual mesh filename=package://mycobot_description/urdf/pro_adaptive_gripper/gri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
- link gripper_right2: geometry collision box size=0.0597 0.0493 0.0200; visual mesh filename=package://mycobot_description/urdf/pro_adaptive_gripper/gri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
- link gripper_right3: geometry collision box size=0.0653 0.0435 0.0086; visual mesh filename=package://mycobot_description/urdf/pro_adaptive_gripper/gri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

Commit message: fix(gazebo): corrige les liens enfants des 3 joints caméra
Les joints world_to_camera_right/left/top référençaient des liens
camera_link_right/left/top inexistants (les liens définis sont
camera_link_1/2/3). robot_state_publisher échouait au parsing URDF
("child link [camera_link_left] not found") et le robot ne se
chargeait pas dans Gazebo. Résidu de la résolution de conflit PR #9
où la version des joints a été gardée sans aligner les noms de liens.

File: mycobot_description/urdf/320_pi/mycobot_pro_320_pi_gazebo.urdf (robot description, URDF)
Before this commit: robot mycobot_320_pi, 19 links, 18 joints
Joints:
- joint world_to_camera_left: child camera_link_left -> camera_link_2
- joint world_to_camera_right: child camera_link_right -> camera_link_1
- joint world_to_camera_top: child camera_link_top -> camera_link_3

Commit message: perf(gazebo): collisions du robot allegees, simulation ~4x plus rapide
Les 14 collisions de mycobot_pro_320_pi_gazebo.urdf reprenaient les DAE
d affichage, 52 000 a 243 000 faces par lien, 1,1 million au total,
qu ODE testait a chaque pas de 1 ms. Les retirer faisait passer la scene
de tri de 0,17 a 0,96 fois le temps reel ; les cameras, elles, ne pesent
presque rien (0,158 -> 0,174 sans elles).

Chaque DAE est remplace par son enveloppe exterieure dans le meme repere
(voxelisee, marching cubes, decimee a 3 000 faces) :
scripts/simplify_collision_meshes.py. Matiere ajoutee p99 <= 1,8 mm sur
le bras, <= 0,62 mm sur les doigts, qui ont 2,5 mm de jeu a la saisie.
Affichage, origines, masses et ..._nogripper.urdf inchanges.

RTF, GPU NVIDIA : 0,17 -> 0,73 sans interface, 0,14 -> 0,62 avec. Tri
perception YOLO : graines 1-4 16/16 au premier essai ; graine 7 avec
interface, DREAM et dashboard 4/4 en 4 min 34 s au lieu de 22 min 14 s.
Graines 5-10 encore a faire avant de conclure contre le 40/40 d Osama.

Depend de fix/tri-yolo-launch pour lancer tri_yolo hors du poste
d origine.

File: mycobot_description/urdf/320_pi/mycobot_pro_320_pi_gazebo.urdf (robot description, URDF)
Before this commit: robot mycobot_320_pi, 15 links, 14 joints
Links:
- link base: geometry collision mesh filename=package://mycobot_description/urdf/320_pi/collision/base.stl scale=0.001 0.001 0.001; visual mesh filename=package://mycobot_description/urdf/320_pi/base.dae
- link gripper_base: geometry collision mesh filename=package://mycobot_description/urdf/pro_adaptive_gripper/col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 scale=0.001 0.001 0.001; visual mesh filename=package://mycobot_description/urdf/pro_adaptive_gripper/gri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
- link gripper_left1: geometry collision mesh filename=package://mycobot_description/urdf/pro_adaptive_gripper/col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 scale=0.001 0.001 0.001; visual mesh filename=package://mycobot_description/urdf/pro_adaptive_gripper/gri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
- link gripper_left2: geometry collision mesh filename=package://mycobot_description/urdf/pro_adaptive_gripper/col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 scale=0.001 0.001 0.001; visual mesh filename=package://mycobot_description/urdf/pro_adaptive_gripper/gri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
- link gripper_left3: geometry collision mesh filename=package://mycobot_description/urdf/pro_adaptive_gripper/col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 scale=0.001 0.001 0.001; visual mesh filename=package://mycobot_description/urdf/pro_adaptive_gripper/gri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
- link gripper_right1: geometry collision mesh filename=package://mycobot_description/urdf/pro_adaptive_gripper/col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 scale=0.001 0.001 0.001; visual mesh filename=package://mycobot_description/urdf/pro_adaptive_gripper/gri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
- link gripper_right2: geometry collision mesh filename=package://mycobot_description/urdf/pro_adaptive_gripper/col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 scale=0.001 0.001 0.001; visual mesh filename=package://mycobot_description/urdf/pro_adaptive_gripper/gri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
- link gripper_right3: geometry collision mesh filename=package://mycobot_description/urdf/pro_adaptive_gripper/col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 scale=0.001 0.001 0.001; visual mesh filename=package://mycobot_description/urdf/pro_adaptive_gripper/gri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
- link link1: geometry collision mesh filename=package://mycobot_description/urdf/320_pi/collision/link1.s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 scale=0.001 0.001 0.001; visual mesh filename=package://mycobot_description/urdf/320_pi/link1.dae
- link link2: geometry collision mesh filename=package://mycobot_description/urdf/320_pi/collision/link2.s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 scale=0.001 0.001 0.001; visual mesh filename=package://mycobot_description/urdf/320_pi/link2.dae
- link link3: geometry collision mesh filename=package://mycobot_description/urdf/320_pi/collision/link3.s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 scale=0.001 0.001 0.001; visual mesh filename=package://mycobot_description/urdf/320_pi/link3.dae
- link link4: geometry collision mesh filename=package://mycobot_description/urdf/320_pi/collision/link4.s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 scale=0.001 0.001 0.001; visual mesh filename=package://mycobot_description/urdf/320_pi/link4.dae
- link link5: geometry collision mesh filename=package://mycobot_description/urdf/320_pi/collision/link5.s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 scale=0.001 0.001 0.001; visual mesh filename=package://mycobot_description/urdf/320_pi/link5.dae
- link link6: geometry collision mesh filename=package://mycobot_description/urdf/320_pi/collision/link6_2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 scale=0.001 0.001 0.001; visual mesh filename=package://mycobot_description/urdf/320_pi/link6_2022.dae
